Commit message: create core components

File: Packo - Modelagem.urdf (robot description, URDF)
Before this commit: robot packo, 10 links, 9 joints
Links:
- added link bottom_drawer; collision box size=0.47 0.46 0.01; visual box size=0.47 0.46 0.01
- added link bottom_drawer_door; collision box size=0.01 0.1825 0.46; visual box size=0.01 0.1825 0.46
- added link bottom_drawer_hinge; collision cylinder length=.46 radius=0.01; visual cylinder length=.46 radius=0.01
- added link front_cover; collision box size=0.02 0.46 0.1825; visual box size=0.02 0.46 0.1825
- added link measurer; collision sphere radius=0.005; visual sphere radius=0.005
- added link middle_drawer; collision box size=0.47 0.46 0.01; visual box size=0.47 0.46 0.01
- added link middle_drawer_door; collision box size=0.01 0.187 0.46; visual box size=0.01 0.187 0.46
- added link middle_drawer_hinge; collision cylinder length=.46 radius=0.01; visual cylinder length=.46 radius=0.01
- added link top_drawer; collision box size=0.47 0.46 0.01; visual box size=0.47 0.46 0.01
- added link top_drawer_divider; collision box size=0.47 0.01 0.1925; visual box size=0.47 0.01 0.1925
- added link top_left_drawer_door; collision box size=0.01 0.1975 0.225; visual box size=0.01 0.1975 0.225
- added link top_left_drawer_hinge; collision cylinder length=.225 radius=0.01; visual cylinder length=.225 radius=0.01
- added link top_right_drawer_door; collision box size=0.01 0.1975 0.225; visual box size=0.01 0.1975 0.225
- added link top_right_drawer_hinge; collision cylinder length=.225 radius=0.01; visual cylinder length=.225 radius=0.01
Joints:
- added joint base_to_bottom_drawer: type fixed, parent base, child bottom_drawer, origin xyz=0 0 0.1975 rpy=0 0 0
- added joint base_to_front_cover: type fixed, parent base, child front_cover, origin xyz=0.24 0 0.10125 rpy=0 0 0
- added joint base_to_middle_drawer: type fixed, parent base, child middle_drawer, origin xyz=0 0 0.385 rpy=0 0 0
- added joint base_to_top_drawer: type fixed, parent base, child top_drawer, origin xyz=0 0 0.5775 rpy=0 0 0
- added joint base_to_top_drawer_divider: type fixed, parent base, child top_drawer_divider, origin xyz=0 0 0.67375 rpy=0 0 0
- added joint bottom_drawer_hinge_to_bottom_drawer_door: type fixed, parent bottom_drawer_hinge, child bottom_drawer_door, origin xyz=0 0.08625 0 rpy=0 0 0
- added joint bottom_drawer_to_bottom_drawer_hinge: type continuous, parent bottom_drawer, child bottom_drawer_hinge, origin xyz=0.23 0 0 rpy=1.57 0 0, axis 0 0 1
- added joint middle_drawer_hinge_to_middle_drawer_door: type fixed, parent middle_drawer_hinge, child middle_drawer_door, origin xyz=0 0.091 0 rpy=0 0 0
- added joint middle_drawer_to_middle_drawer_hinge: type continuous, parent middle_drawer, child middle_drawer_hinge, origin xyz=0.23 0 0 rpy=1.57 0 0, axis 0 0 1
- added joint top_drawer_to_top_left_drawer_hinge: type continuous, parent top_drawer, child top_left_drawer_hinge, origin xyz=0.23 -0.1175 0 rpy=1.57 0 0, axis 0 0 1
- added joint top_drawer_to_top_right_drawer_hinge: type continuous, parent top_drawer, child top_right_drawer_hinge, origin xyz=0.23 0.1175 0 rpy=1.57 0 0, axis 0 0 1
- added joint top_left_drawer_hinge_to_top_left_drawer_door: type fixed, parent top_left_drawer_hinge, child top_left_drawer_door, origin xyz=0 0.0935 0 rpy=0 0 0
- added joint top_right_drawer_hinge_to_top_right_drawer_door: type fixed, parent top_right_drawer_hinge, child top_right_drawer_door, origin xyz=0 0.0935 0 rpy=0 0 0

Commit message: add screen

File: Packo - Modelagem.urdf (robot description, URDF)
Before this commit: robot packo, 24 links, 22 joints
Links:
- removed link measurer
- added link screen; collision box size=0.01 0.2 0.1; visual box size=0.01 0.2 0.1
- added link screen_base; collision cylinder length=.05 radius=0.22; visual cylinder length=.05 radius=0.22
Joints:
- added joint screen_base_to_screen: type fixed, parent screen_base, child screen, origin xyz=0.20 0 0.07 rpy=0 -0.35 0
- added joint top_wall_to_screen_base: type continuous, parent top_wall, child screen_base, origin xyz=0 0 0.02 rpy=0 0 0, axis 0 0 1

Commit message: add inertial tags

File: Packo - Modelagem.urdf (robot description, URDF)
Before this commit: robot packo, 25 links, 24 joints
Links:
- link back_wall: mass None -> 0.4
- link base: mass None -> 5
- link bottom_drawer: mass None -> 0.1
- link bottom_drawer_door: mass None -> 0.05
- link bottom_drawer_hinge: mass None -> 0.005
- link front_cover: mass None -> 0.2
- link left_back_wheel: mass None -> 2
- link left_front_wheel: mass None -> 2
- link left_wall: mass None -> 0.4
- link middle_drawer: mass None -> 0.1
- link middle_drawer_door: mass None -> 0.05
- link middle_drawer_hinge: mass None -> 0.005
- link right_back_wheel: mass None -> 2
- link right_front_wheel: mass None -> 2
- link right_wall: mass None -> 0.4
- link screen: mass None -> 0.1
- link screen_base: mass None -> 2
- link top_drawer: mass None -> 0.1
- link top_drawer_divider: mass None -> 0.2
- link top_left_drawer_door: mass None -> 0.05
- link top_left_drawer_hinge: mass None -> 0.005
- link top_right_drawer_door: mass None -> 0.05
- link top_right_drawer_hinge: mass None -> 0.005
- link top_wall: mass None -> 0.4

Commit message: update modeling

File: Packo - Modelagem.urdf (robot description, URDF)
Before this commit: robot packo, 25 links, 24 joints
Links:
- link base: mass 5 -> 10
- link screen_base: mass 2 -> 0.2
